File: homeassistant-temp-sensor-pcb/homeassistant-temp-sensor-pcb.kicad_pcb (KiCad board)
At the start: 0 parts

Commit message: schematic
Parts:
- added U1: WeMos_mini, wemos_d1_mini:D1_mini_board, F.Cu at (149.9, 96.5)
- added U2: DHT11, Sensor:Aosong_DHT11_5.5x12.0_P2.54mm, F.Cu at (166.9, 80.9)
Other:
- copper layers 0 -> 2

Commit message: more pcb
Parts:
- removed U2: DHT11, Sensor:Aosong_DHT11_5.5x12.0_P2.54mm
- added J1: Conn_01x01_Pin, Connector_PinHeader_2.54mm:PinHeader_1x01_P2.54mm_Vertical, F.Cu at (152.4, 101.0)
- added J2: Conn_01x01_Pin, Connector_PinHeader_2.54mm:PinHeader_1x01_P2.54mm_Vertical, F.Cu at (147.3, 101.0)
- added U3: DHT11, Connector_PinHeader_2.54mm:PinHeader_1x03_P2.54mm_Vertical, F.Cu at (147.3, 104.1)
Connections:
- U1 pad 2: Net-(U1-GND) -> GND
Routing:
- net Net-(U1-D4): track 0.00 -> 15.4 mm
- net Net-(U1-5V): track 0.00 -> 8.89 mm
- added copper zone on F.Cu, net GND
Other:
- board outline added: 26.7 x 8.9 mm
